Commit message: feat(ros2): set up ros2 description and sim packages

File: ros2_ws/src/bot_description/urdf/quad_quad_limb.urdf (robot description, URDF)
Before this commit: robot fixed_limb_test, 6 links, 5 joints
Links:
- link base_link: geometry collision mesh filename=package://bot_description/meshes/base_link.STL; visual mesh filename=package://bot_description/meshes/base_link.STL
- link femur_link: geometry collision mesh filename=package://bot_description/meshes/femur_link.STL; visual mesh filename=package://bot_description/meshes/femur_link.STL
- link rod_link: geometry collision mesh filename=package://bot_description/meshes/rod_link.STL; visual mesh filename=package://bot_description/meshes/rod_link.STL
- link shoulder_link: geometry collision mesh filename=package://bot_description/meshes/shoulder_link.STL; visual mesh filename=package://bot_description/meshes/shoulder_link.STL
- link tab_link: geometry collision mesh filename=package://bot_description/meshes/tab_link.STL; visual mesh filename=package://bot_description/meshes/tab_link.STL
- link tibia_link: geometry collision mesh filename=package://bot_description/meshes/tibia_link.STL; visual mesh filename=package://bot_description/meshes/tibia_link.STL

Commit message: bug(urdf): rotate haa joint by pi rads

File: ros2_ws/src/bot_description/urdf/quad_quad_limb.urdf (robot description, URDF)
Before this commit: robot quad_quad_limb, 6 links, 5 joints
Joints:
- joint haa_joint: origin xyz=-0.001 0.006 -0.016 rpy=3.1416 -1.5708 0 -> xyz=-0.001 0.006 -0.016 rpy=0 -1.5708 0

Commit message: urdf: rescale inertias and add effort values to joints

File: ros2_ws/src/bot_description/urdf/quad_quad_limb.urdf (robot description, URDF)
Before this commit: robot quad_quad_limb, 6 links, 5 joints
Links:
- link base_link: mass 0.00723402556361831 -> 0.723402556361831
- link femur_link: mass 0.0138239022547814 -> 1.38239022547814
- link rod_link: mass 0.000929490166689096 -> 0.0929490166689096
- link shoulder_link: mass 0.0148104574438063 -> 1.48104574438063
- link tab_link: mass 0.00116134718742782 -> 0.116134718742782
- link tibia_link: mass 0.0070755567397191 -> 0.70755567397191
Joints:
- joint haa_joint: limit lower=-1.5708 upper=0 effort=0 velocity=0 -> lower=-1.5708 upper=0 effort=58.8 velocity=5.0
- joint hfe_joint: limit lower=0 upper=3.14 effort=0 velocity=0 -> lower=0 upper=3.14 effort=58.8 velocity=5.0
- joint kfe_motor_joint: limit lower=-0.87267 upper=0.87267 effort=0 velocity=0 -> lower=-0.87267 upper=0.87267 effort=58.8 velocity=5.0
- joint knee_joint: limit lower=-0.87267 upper=0.87267 effort=0 velocity=0 -> lower=-0.87267 upper=0.87267 effort=1000.0 velocity=5.0
- joint rod_joint: limit lower=-0.87267 upper=0.87267 effort=0 velocity=0 -> lower=-0.87267 upper=0.87267 effort=1000.0 velocity=5.0
