Commit message: feat(urdf): integrate ros2_control into limb urdf

File: ros2_ws/src/bot_description/urdf/quad_quad_limb.urdf.xacro (robot description, xacro)
@@ -170,3 +170,28 @@
         <limit lower="-0.87267" upper="0.87267" effort="1000.0" velocity="5.0" />
     </joint>
+    <ros2_control name="GazeboSystem" type="system">
+        <hardware>
+            <plugin>gz_ros2_control/GazeboSimSystem</plugin>
+        </hardware>
+        <joint name="haa_joint">
+            <command_interface name="position"/>
+            <state_interface name="position"/>
+            <state_interface name="velocity"/>
+        </joint>
+        <joint name="hfe_joint">
+            <command_interface name="position"/>
+            <state_interface name="position"/>
+            <state_interface name="velocity"/>
+        </joint>
+        <joint name="knee_joint">
+            <command_interface name="position"/>
+            <state_interface name="position"/>
+            <state_interface name="velocity"/>
+        </joint>
+    </ros2_control>
+    <gazebo>
+        <plugin filename="gz_ros2_control-system" name="gz_ros2_control::GazeboSimROS2ControlPlugin">
+            <parameters>$(find bot_control)/config/controllers.yaml</parameters>
+        </plugin>
+    </gazebo>
 </robot>

Commit message: feat(urdf): anchor limb to world link

File: ros2_ws/src/bot_description/urdf/quad_quad_limb.urdf.xacro (robot description, xacro)
@@ -2,4 +2,5 @@
 <robot name="quad_quad_limb">
     <!-- Links -->
+    <link name="world" />
     <link name="base_link">
         <inertial>
@@ -135,4 +136,9 @@
     </link>
     <!-- Joints -->
+    <joint name="world_fixed" type="fixed">
+        <origin xyz="0 0 0.2" rpy="-1.5708 0 1.5708"/>
+        <parent link="world"/>
+        <child link="base_link"/>
+    </joint>
     <joint name="haa_joint" type="revolute">
         <origin xyz="-0.001 0.006 -0.016" rpy="0 -1.5708 0" />

Commit message: fix(ros/urdf): adjust haa and hfe bounds to prevent limit sticking

File: ros2_ws/src/bot_description/urdf/quad_quad_limb.urdf.xacro (robot description, xacro)
@@ -146,5 +146,5 @@
         <child link="shoulder_link" />
         <axis xyz="0 0 1" />
-        <limit lower="-1.5708" upper="0" effort="58.8" velocity="5.0" />
+        <limit lower="-0.5236" upper="0.5236" effort="1000.0" velocity="5.0" />
     </joint>
     <joint name="hfe_joint" type="revolute">
@@ -152,6 +152,6 @@
         <parent link="shoulder_link" />
         <child link="femur_link" />
-        <axis xyz="0 0 -1" />
-        <limit lower="0" upper="3.14" effort="58.8" velocity="5.0" />
+        <axis xyz="0 0 1" />
+        <limit lower="-1.5708" upper="1.5708" effort="1000.0" velocity="5.0" />
     </joint>
     <joint name="knee_joint" type="revolute">
@@ -167,5 +167,5 @@
         <child link="tab_link" />
         <axis xyz="0 0 -1" />
-        <limit lower="-0.87267" upper="0.87267" effort="58.8" velocity="5.0" />
+        <limit lower="-0.87267" upper="0.87267" effort="1000.0" velocity="5.0" />
     </joint>
     <joint name="rod_joint" type="revolute">

Commit message: feat(ros/bot_gate): init command gait pkg

File: ros2_ws/src/bot_description/urdf/quad_quad_limb.urdf.xacro (robot description, xacro)
@@ -146,5 +146,5 @@
         <child link="shoulder_link" />
         <axis xyz="0 0 1" />
-        <limit lower="-0.5236" upper="0.5236" effort="1000.0" velocity="5.0" />
+        <limit lower="-3" upper="3" effort="1000.0" velocity="5.0" />
     </joint>
     <joint name="hfe_joint" type="revolute">
@@ -153,5 +153,5 @@
         <child link="femur_link" />
         <axis xyz="0 0 1" />
-        <limit lower="-1.5708" upper="1.5708" effort="1000.0" velocity="5.0" />
+        <limit lower="-3" upper="3" effort="1000.0" velocity="5.0" />
     </joint>
     <joint name="knee_joint" type="revolute">
@@ -160,5 +160,5 @@
         <child link="tibia_link" />
         <axis xyz="0 0 1" />
-        <limit lower="-0.87267" upper="0.87267" effort="1000.0" velocity="5.0" />
+        <limit lower="-3" upper="3" effort="1000.0" velocity="5.0" />
     </joint>
     <joint name="kfe_motor_joint" type="revolute">
@@ -167,5 +167,5 @@
         <child link="tab_link" />
         <axis xyz="0 0 -1" />
-        <limit lower="-0.87267" upper="0.87267" effort="1000.0" velocity="5.0" />
+        <limit lower="-3" upper="3" effort="1000.0" velocity="5.0" />
     </joint>
     <joint name="rod_joint" type="revolute">
@@ -174,5 +174,5 @@
         <child link="rod_link" />
         <axis xyz="0 0 -1" />
-        <limit lower="-0.87267" upper="0.87267" effort="1000.0" velocity="5.0" />
+        <limit lower="-3" upper="3" effort="1000.0" velocity="5.0" />
     </joint>
     <ros2_control name="GazeboSystem" type="system">
@@ -182,6 +182,6 @@
         <joint name="haa_joint">
             <command_interface name="position">
-                <param name="min">-0.5236</param>
-                <param name="max">0.5236</param>
+                <param name="min">-3</param>
+                <param name="max">3</param>
             </command_interface>
             <state_interface name="position">
@@ -193,6 +193,6 @@
         <joint name="hfe_joint">
             <command_interface name="position">
-                <param name="min">-1.5708</param>
-                <param name="max">1.5708</param>
+                <param name="min">-3</param>
+                <param name="max">3</param>
             </command_interface>
             <state_interface name="position">
@@ -204,6 +204,6 @@
         <joint name="knee_joint">
             <command_interface name="position">
-                <param name="min">-0.87267</param>
-                <param name="max">0.87267</param>
+                <param name="min">-3</param>
+                <param name="max">3</param>
             </command_interface>
             <state_interface name="position">
