Commit message: feat(ros/urdf): pass motor params to ros2_control

File: ros2_ws/src/bot_description/urdf/robot.urdf.xacro (robot description, xacro)
@@ -23,5 +23,4 @@
     <xacro:limb prefix="bl" x="${-leg_x}" y="${leg_y}"  z="${leg_z}" r="${leg_roll}" p="${leg_pitch}" yw="${leg_yaw}"  inverted_shoulder="true"  hfe_axis_mult="-1" kfe_axis_mult="-1"/>
     <xacro:limb prefix="br" x="${-leg_x}" y="${-leg_y}" z="${leg_z}" r="${leg_roll}" p="${leg_pitch}" yw="${-leg_yaw}" inverted_shoulder="false" hfe_axis_mult="1" kfe_axis_mult="1"/>
-     macros specific to sim/hardware modes
     <xacro:if value="$(arg sim)">
         <xacro:ros2_control name="GazeboSystem" hardware_plugin="gz_ros2_control/GazeboSimSystem"/>
@@ -29,5 +28,6 @@
     </xacro:if>
     <xacro:unless value="$(arg sim)">
-        <xacro:ros2_control name="HardwareSystem" hardware_plugin="$(arg hardware_plugin)"/>
+        <xacro:ros2_control name="HardwareSystem" hardware_plugin="$(arg hardware_plugin)"
+            motor_params_path="$(find bot_hardware)/config/motor_params.yaml"/>
     </xacro:unless>
 </robot>

File: ros2_ws/src/bot_description/urdf/ros2_control.urdf.xacro (robot description, xacro)
@@ -18,8 +18,12 @@
     </xacro:macro>
     <!-- Ros 2 Control Macro with all joints -->
-    <xacro:macro name="ros2_control" params="name hardware_plugin">
+    <!-- motor_params_path: only set for real hardware; empty for sim -->
+    <xacro:macro name="ros2_control" params="name hardware_plugin motor_params_path:=''">
         <ros2_control name="${name}" type="system">
             <hardware>
                 <plugin>${hardware_plugin}</plugin>
+                <xacro:if value="${motor_params_path != ''}">
+                    <param name="motor_params_path">${motor_params_path}</param>
+                </xacro:if>
             </hardware>
             <xacro:_ros2_control_joint joint_name="fr_haa_joint" lower="${limits['haa']['lower']}"

Commit message: chore(ros/bot_description): pass hardware info through xacro params as oppose to parsing yaml

File: ros2_ws/src/bot_description/urdf/robot.urdf.xacro (robot description, xacro)
@@ -24,10 +24,9 @@
     <xacro:limb prefix="br" x="${-leg_x}" y="${-leg_y}" z="${leg_z}" r="${leg_roll}" p="${leg_pitch}" yw="${-leg_yaw}" inverted_shoulder="false" hfe_axis_mult="1" kfe_axis_mult="1"/>
     <xacro:if value="$(arg sim)">
-        <xacro:ros2_control name="GazeboSystem" hardware_plugin="gz_ros2_control/GazeboSimSystem"/>
+        <xacro:ros2_control name="GazeboSystem" hardware_plugin="gz_ros2_control/GazeboSimSystem" is_hardware="false"/>
         <xacro:gazebo_ros2_control/>
     </xacro:if>
     <xacro:unless value="$(arg sim)">
-        <xacro:ros2_control name="HardwareSystem" hardware_plugin="$(arg hardware_plugin)"
-            motor_params_path="$(find bot_hardware)/config/motor_params.yaml"/>
+        <xacro:ros2_control name="HardwareSystem" hardware_plugin="$(arg hardware_plugin)" is_hardware="true"/>
     </xacro:unless>
 </robot>

File: ros2_ws/src/bot_description/urdf/ros2_control.urdf.xacro (robot description, xacro)
@@ -1,8 +1,9 @@
 <?xml version="1.0"?>
 <robot xmlns:xacro="http://www.ros.org/wiki/xacro" name="ros2_control">
-    <!-- Joint limits loaded from YAML -->
+    <!-- Joint limits and hardware info loaded from YAML -->
     <xacro:property name="limits" value="${xacro.load_yaml('$(find bot_description)/config/joint_limits.yaml')}"/>
+    <xacro:property name="motors" value="${xacro.load_yaml('$(find bot_description)/config/motor_params.yaml')}"/>
     <!-- Single ros2 control joint -->
-    <xacro:macro name="_ros2_control_joint" params="joint_name lower upper initial:=0.0">
+    <xacro:macro name="_ros2_control_joint" params="joint_name lower upper initial:=0.0 is_hardware:=false">
         <joint name="${joint_name}">
             <command_interface name="position">
@@ -15,40 +16,48 @@
             <state_interface name="velocity"/>
             <state_interface name="effort"/>
+            <!-- Additional params of physical motors if running hardware version -->
+            <xacro:if value="${is_hardware}">
+                <param name="motor_id">${motors['joints'][joint_name]['motor_id']}</param>
+                <param name="direction">${motors['joints'][joint_name]['direction']}</param>
+                <param name="offset_ticks">${motors['joints'][joint_name]['offset_ticks']}</param>
+            </xacro:if>
         </joint>
     </xacro:macro>
     <!-- Ros 2 Control Macro with all joints -->
-    <!-- motor_params_path: only set for real hardware; empty for sim -->
-    <xacro:macro name="ros2_control" params="name hardware_plugin motor_params_path:=''">
+    <xacro:macro name="ros2_control" params="name hardware_plugin is_hardware:=false">
         <ros2_control name="${name}" type="system">
             <hardware>
                 <plugin>${hardware_plugin}</plugin>
-                <xacro:if value="${motor_params_path != ''}">
-                    <param name="motor_params_path">${motor_params_path}</param>
+                <xacro:if value="${is_hardware}">
+                    <param name="serial_port">${motors['bus']['serial_port']}</param>
+                    <param name="baud_rate">${motors['bus']['baud_rate']}</param>
+                    <param name="max_velocity_rad_per_s">${motors['bus']['max_velocity_rad_per_s']}</param>
+                    <param name="servo_speed_units">${motors['bus']['servo_speed_units']}</param>
                 </xacro:if>
             </hardware>
             <xacro:_ros2_control_joint joint_name="fr_haa_joint" lower="${limits['haa']['lower']}"
-                                       upper="${limits['haa']['upper']}"/>
+                                       upper="${limits['haa']['upper']}" is_hardware="${is_hardware}"/>
             <xacro:_ros2_control_joint joint_name="fr_hfe_joint" lower="${limits['hfe']['lower']}"
-                                       upper="${limits['hfe']['upper']}"/>
+                                       upper="${limits['hfe']['upper']}" is_hardware="${is_hardware}"/>
             <xacro:_ros2_control_joint joint_name="fr_kfe_joint" lower="${limits['kfe']['lower']}"
-                                       upper="${limits['kfe']['upper']}"/>
+                                       upper="${limits['kfe']['upper']}" is_hardware="${is_hardware}"/>
             <xacro:_ros2_control_joint joint_name="fl_haa_joint" lower="${limits['haa']['lower']}"
-                                       upper="${limits['haa']['upper']}"/>
+                                       upper="${limits['haa']['upper']}" is_hardware="${is_hardware}"/>
             <xacro:_ros2_control_joint joint_name="fl_hfe_joint" lower="${limits['hfe']['lower']}"
-                                       upper="${limits['hfe']['upper']}"/>
+                                       upper="${limits['hfe']['upper']}" is_hardware="${is_hardware}"/>
             <xacro:_ros2_control_joint joint_name="fl_kfe_joint" lower="${limits['kfe']['lower']}"
-                                       upper="${limits['kfe']['upper']}"/>
+                                       upper="${limits['kfe']['upper']}" is_hardware="${is_hardware}"/>
             <xacro:_ros2_control_joint joint_name="br_haa_joint" lower="${limits['haa']['lower']}"
-                                       upper="${limits['haa']['upper']}"/>
+                                       upper="${limits['haa']['upper']}" is_hardware="${is_hardware}"/>
             <xacro:_ros2_control_joint joint_name="br_hfe_joint" lower="${limits['hfe']['lower']}"
-                                       upper="${limits['hfe']['upper']}"/>
+                                       upper="${limits['hfe']['upper']}" is_hardware="${is_hardware}"/>
             <xacro:_ros2_control_joint joint_name="br_kfe_joint" lower="${limits['kfe']['lower']}"
-                                       upper="${limits['kfe']['upper']}"/>
+                                       upper="${limits['kfe']['upper']}" is_hardware="${is_hardware}"/>
             <xacro:_ros2_control_joint joint_name="bl_haa_joint" lower="${limits['haa']['lower']}"
-                                       upper="${limits['haa']['upper']}"/>
+                                       upper="${limits['haa']['upper']}" is_hardware="${is_hardware}"/>
             <xacro:_ros2_control_joint joint_name="bl_hfe_joint" lower="${limits['hfe']['lower']}"
-                                       upper="${limits['hfe']['upper']}"/>
+                                       upper="${limits['hfe']['upper']}" is_hardware="${is_hardware}"/>
             <xacro:_ros2_control_joint joint_name="bl_kfe_joint" lower="${limits['kfe']['lower']}"
-                                       upper="${limits['kfe']['upper']}"/>
+                                       upper="${limits['kfe']['upper']}" is_hardware="${is_hardware}"/>
         </ros2_control>
     </xacro:macro>
