Commit message: style(urdf): add visual materials for parts

File: ros2_ws/src/bot_description/urdf/body.urdf.xacro (robot description, xacro)
@@ -16,4 +16,7 @@
                     <mesh filename="package://bot_description/meshes/body.STL"/>
                 </geometry>
+                <material name="body_plastic">
+                    <color rgba="0.65 0.70 0.75 1.0"/>
+                </material>
             </visual>
             <collision>

File: ros2_ws/src/bot_description/urdf/limb.urdf.xacro (robot description, xacro)
@@ -19,4 +19,7 @@
                     <mesh filename="package://bot_description/meshes/haa_horn.STL" scale="1 1 1"/>
                 </geometry>
+                <material name="joint_horn_accent">
+                    <color rgba="0.95 0.65 0.20 1.0"/>
+                </material>
             </visual>
             <visual>
@@ -25,4 +28,7 @@
                     <mesh filename="package://bot_description/meshes/shoulder_casing.STL" scale="1 1 1"/>
                 </geometry>
+                <material name="shoulder_plastic">
+                    <color rgba="0.55 0.62 0.72 1.0"/>
+                </material>
             </visual>
             <visual>
@@ -31,4 +37,7 @@
                     <mesh filename="package://bot_description/meshes/hfe_servo.STL" scale="1 1 1"/>
                 </geometry>
+                <material name="motor_dark_gray">
+                    <color rgba="0.20 0.20 0.22 1.0"/>
+                </material>
             </visual>
             <collision>
@@ -63,4 +72,7 @@
                     <mesh filename="package://bot_description/meshes/hfe_horn.STL" scale="1 1 1"/>
                 </geometry>
+                <material name="joint_horn_accent">
+                    <color rgba="0.95 0.65 0.20 1.0"/>
+                </material>
             </visual>
             <visual>
@@ -69,4 +81,7 @@
                     <mesh filename="package://bot_description/meshes/femur.STL" scale="1 1 1"/>
                 </geometry>
+                <material name="femur_plastic">
+                    <color rgba="0.52 0.69 0.84 1.0"/>
+                </material>
             </visual>
             <visual>
@@ -75,4 +90,7 @@
                     <mesh filename="package://bot_description/meshes/kfe_servo.STL" scale="1 1 1"/>
                 </geometry>
+                <material name="motor_dark_gray">
+                    <color rgba="0.20 0.20 0.22 1.0"/>
+                </material>
             </visual>
             <collision>
@@ -107,4 +125,7 @@
                     <mesh filename="package://bot_description/meshes/tibia.STL" scale="1 1 1"/>
                 </geometry>
+                <material name="tibia_plastic">
+                    <color rgba="0.56 0.78 0.62 1.0"/>
+                </material>
             </visual>
             <collision>

Commit message: feat(urdf): update urdf settings from new export

File: ros2_ws/src/bot_description/urdf/body.urdf.xacro (robot description, xacro)
@@ -6,24 +6,24 @@
         <link name="body_link">
             <inertial>
-                <origin xyz="0.0003026 -0.033305 -0.00066994" rpy="0 0 0"/>
-                <mass value="0.33425"/>
-                <inertia ixx="0.00022631" ixy="1.6841E-06" ixz="2.4325E-07" iyy="0.00068307" iyz="-2.2508E-06"
-                         izz="0.00051261"/>
-            </inertial>
-            <visual>
-                <origin xyz="0 0 0" rpy="0 0 0"/>
-                <geometry>
-                    <mesh filename="package://bot_description/meshes/body.STL"/>
-                </geometry>
-                <material name="body_plastic">
-                    <color rgba="0.65 0.70 0.75 1.0"/>
-                </material>
-            </visual>
-            <collision>
-                <origin xyz="0 0 0" rpy="0 0 0"/>
-                <geometry>
-                    <mesh filename="package://bot_description/meshes/body.STL"/>
-                </geometry>
-            </collision>
+                    <origin xyz="0.010253 -0.021653 -0.00076856" rpy="0 0 0" />
+                    <mass value="0.60969" />
+                    <inertia ixx="0.00097469" ixy="7.6657E-05" ixz="5.131E-06" iyy="0.0038736" iyz="-2.4748E-06"
+                             izz="0.0031856" />
+                </inertial>
+                <visual>
+                    <origin xyz="0 0 0" rpy="0 0 0" />
+                    <geometry>
+                        <mesh filename="package://chassis_sub.SLDASM/meshes/chassis_link.STL" />
+                    </geometry>
+                    <material name="">
+                        <color rgba="0.5451 0.61569 0.85882 1" />
+                    </material>
+                </visual>
+                <collision>
+                    <origin xyz="0 0 0" rpy="0 0 0" />
+                    <geometry>
+                        <mesh filename="package://bot_description/meshes/chassis_link.STL" />
+                    </geometry>
+                </collision>
         </link>
         <!-- Joints -->
@@ -31,5 +31,5 @@
             <parent link="base_link"/>
             <child link="body_link"/>
-            <origin xyz="0 0 0" rpy="-1.5708 0 0"/>
+            <origin xyz="0 0 0" rpy="0 0 0"/>
         </joint>
     </xacro:macro>

File: ros2_ws/src/bot_description/urdf/limb.urdf.xacro (robot description, xacro)
@@ -9,34 +9,16 @@
         <link name="${prefix}shoulder_link">
             <inertial>
-                <origin xyz="0.018766 0.016329 0.0079907" rpy="0 0 0"/>
-                <mass value="0.01481"/>
-                <inertia ixx="1.3996E-06" ixy="-1.6833E-08" ixz="-7.906E-10" iyy="1.8819E-06" iyz="-3.0123E-10"
-                         izz="2.5913E-06"/>
+                <origin xyz="0.00123926352361432 0.00335245027216135 0.020963936804564" rpy="0 0 0" />
+                <mass value="0.0703942212311305" />
+                <inertia ixx="2.76576288052366E-05" ixy="-1.39471839648609E-07" ixz="-2.88488463706858E-07"
+                         iyy="1.71370747114446E-05" iyz="-6.19746545161347E-08" izz="2.60685249875832E-05" />
             </inertial>
             <visual>
                 <origin xyz="0 0 0" rpy="0 0 0"/>
                 <geometry>
-                    <mesh filename="package://bot_description/meshes/haa_horn.STL" scale="1 1 1"/>
+                    <mesh filename="package://bot_description/meshes/shoulder_link.STL" />
                 </geometry>
-                <material name="joint_horn_accent">
-                    <color rgba="0.95 0.65 0.20 1.0"/>
-                </material>
-            </visual>
-            <visual>
-                <origin xyz="0 0 0" rpy="0 0 0"/>
-                <geometry>
-                    <mesh filename="package://bot_description/meshes/shoulder_casing.STL" scale="1 1 1"/>
-                </geometry>
-                <material name="shoulder_plastic">
-                    <color rgba="0.55 0.62 0.72 1.0"/>
-                </material>
-            </visual>
-            <visual>
-                <origin xyz="0 0 0" rpy="0 0 0"/>
-                <geometry>
-                    <mesh filename="package://bot_description/meshes/hfe_servo.STL" scale="1 1 1"/>
-                </geometry>
-                <material name="motor_dark_gray">
-                    <color rgba="0.20 0.20 0.22 1.0"/>
+                <material name="">
+                    <color rgba="0.792156862745098 0.819607843137255 0.933333333333333 1" />
                 </material>
             </visual>
@@ -44,17 +26,5 @@
                 <origin xyz="0 0 0" rpy="0 0 0"/>
                 <geometry>
-                    <mesh filename="package://bot_description/meshes/haa_horn.STL" scale="1 1 1"/>
-                </geometry>
-            </collision>
-            <collision>
-                <origin xyz="0 0 0" rpy="0 0 0"/>
-                <geometry>
-                    <mesh filename="package://bot_description/meshes/shoulder_casing.STL" scale="1 1 1"/>
-                </geometry>
-            </collision>
-            <collision>
-                <origin xyz="0 0 0" rpy="0 0 0"/>
-                <geometry>
-                    <mesh filename="package://bot_description/meshes/hfe_servo.STL" scale="1 1 1"/>
+                    <mesh filename="package://bot_description/meshes/shoulder_link.STL" scale="1 1 1"/>
                 </geometry>
             </collision>
@@ -62,34 +32,39 @@
         <link name="${prefix}femur_link">
             <inertial>
-                <origin xyz="0.012387 -0.00071898 0.017314" rpy="0 0 0"/>
-                <mass value="0.015915"/>
-                <inertia ixx="9.3139E-07" ixy="-7.9194E-10" ixz="-9.4792E-08" iyy="3.7356E-06" iyz="1.3143E-09"
-                         izz="3.3585E-06"/>
+                <origin xyz="0.0219749723740116 1.10674379296058E-05 0.0317318417810033" rpy="0 0 0" />
+                <mass value="0.0578650759594537" />
+                <inertia ixx="7.21606846133888E-06" ixy="-2.43047276138592E-09" ixz="-8.71808476080296E-07"
+                         iyy="3.86361231869082E-05" iyz="-9.13958901614113E-10" izz="3.73315278091681E-05" />
             </inertial>
             <visual>
-                <origin xyz="0 0 0" rpy="0 0 0"/>
+                <origin xyz="0 0 0" rpy="0 0 0" />
                 <geometry>
-                    <mesh filename="package://bot_description/meshes/hfe_horn.STL" scale="1 1 1"/>
+                    <mesh filename="package://bot_description/meshes/femur_link.STL" />
                 </geometry>
-                <material name="joint_horn_accent">
-                    <color rgba="0.95 0.65 0.20 1.0"/>
+                <material name="">
+                    <color rgba="0.96078431372549 0.96078431372549 0.964705882352941 1" />
                 </material>
             </visual>
+            <collision>
+                <origin xyz="0 0 0" rpy="0 0 0" />
+                <geometry>
+                    <mesh filename="package://bot_description/meshes/femur_link.STL" />
+                </geometry>
+            </collision>
+        </link>
+        <link name="${prefix}tibia_link">
+            <inertial>
+                <origin xyz="0.031878867699759 5.86889321863016E-11 1.81508030133726E-08" rpy="0 0 0" />
+                <mass value="0.0109091234821787" />
+                <inertia ixx="1.95526217620308E-07" ixy="1.4570117043835E-11" ixz="1.85497777908555E-11"
+                         iyy="1.01874475115624E-05" iyz="-4.19910780669847E-12" izz="1.01972686884836E-05" />
+            </inertial>
             <visual>
-                <origin xyz="0 0 0" rpy="0 0 0"/>
+                <origin xyz="0 0 0" rpy="0 0 0" />
                 <geometry>
-                    <mesh filename="package://bot_description/meshes/femur.STL" scale="1 1 1"/>
+                    <mesh filename="package://bot_description/meshes/tibia_link.STL" />
                 </geometry>
-                <material name="femur_plastic">
-                    <color rgba="0.52 0.69 0.84 1.0"/>
-                </material>
-            </visual>
-            <visual>
-                <origin xyz="0 0 0" rpy="0 0 0"/>
-                <geometry>
-                    <mesh filename="package://bot_description/meshes/kfe_servo.STL" scale="1 1 1"/>
-                </geometry>
-                <material name="motor_dark_gray">
-                    <color rgba="0.20 0.20 0.22 1.0"/>
+                <material name="">
+                    <color rgba="0.545098039215686 0.615686274509804 0.858823529411765 1" />
                 </material>
             </visual>
@@ -97,40 +72,5 @@
                 <origin xyz="0 0 0" rpy="0 0 0"/>
                 <geometry>
-                    <mesh filename="package://bot_description/meshes/hfe_horn.STL" scale="1 1 1"/>
-                </geometry>
-            </collision>
-            <collision>
-                <origin xyz="0 0 0" rpy="0 0 0"/>
-                <geometry>
-                    <mesh filename="package://bot_description/meshes/femur.STL" scale="1 1 1"/>
-                </geometry>
-            </collision>
-            <collision>
-                <origin xyz="0 0 0" rpy="0 0 0"/>
-                <geometry>
-                    <mesh filename="package://bot_description/meshes/kfe_servo.STL" scale="1 1 1"/>
-                </geometry>
-            </collision>
-        </link>
-        <link name="${prefix}tibia_link">
-            <inertial>
-                <origin xyz="0.0019117 0.036934 -0.0058072" rpy="0 0 0"/>
-                <mass value="0.052333"/>
-                <inertia ixx="3.6178E-05" ixy="3.873E-06" ixz="-6.0786E-07" iyy="2.0314E-05" iyz="6.2224E-06"
-                         izz="2.4513E-05"/>
-            </inertial>
-            <visual>
-                <origin xyz="0 0 0" rpy="0 0 0"/>
-                <geometry>
-                    <mesh filename="package://bot_description/meshes/tibia.STL" scale="1 1 1"/>
-                </geometry>
-                <material name="tibia_plastic">
-                    <color rgba="0.56 0.78 0.62 1.0"/>
-                </material>
-            </visual>
-            <collision>
-                <origin xyz="0 0 0" rpy="0 0 0"/>
-                <geometry>
-                    <mesh filename="package://bot_description/meshes/tibia.STL" scale="1 1 1"/>
+                    <mesh filename="package://bot_description/meshes/tibia_link.STL" scale="1 1 1"/>
                 </geometry>
             </collision>

File: ros2_ws/src/bot_description/urdf/robot.urdf.xacro (robot description, xacro)
@@ -6,7 +6,7 @@
     <xacro:arg name="hardware_plugin" default="mock_components/GenericSystem"/>
     <!-- Common leg placement/orientation values -->
-    <xacro:property name="leg_x" value="0.0765"/>
-    <xacro:property name="leg_y" value="-0.009"/>
-    <xacro:property name="leg_z" value="0.0338"/>
+    <xacro:property name="leg_x" value="-0.04991"/>
+    <xacro:property name="leg_y" value="-0.0056409"/>
+    <xacro:property name="leg_z" value="-0.066876"/>
     <xacro:property name="leg_pitch" value="1.5708"/>
     <xacro:property name="leg_roll_flip" value="3.1416"/>

Commit message: feat(urdf): integrate into xacro strcuture new robot casing and two limbs

File: ros2_ws/src/bot_description/urdf/body.urdf.xacro (robot description, xacro)
@@ -6,16 +6,16 @@
         <link name="body_link">
             <inertial>
-                    <origin xyz="0.010253 -0.021653 -0.00076856" rpy="0 0 0" />
-                    <mass value="0.60969" />
-                    <inertia ixx="0.00097469" ixy="7.6657E-05" ixz="5.131E-06" iyy="0.0038736" iyz="-2.4748E-06"
-                             izz="0.0031856" />
+                    <origin xyz="-0.000889242251136346 0.00065866860454622 0.0252390940732559" rpy="0 0 0" />
+                    <mass value="0.482255179604208" />
+                    <inertia ixx="0.000590030011142084" ixy="1.74833019226649E-07" ixz="1.21790430692212E-05"
+                             iyy="0.000652273135047948" iyz="5.42047268018053E-08" izz="0.000968313234449169" />
                 </inertial>
                 <visual>
                     <origin xyz="0 0 0" rpy="0 0 0" />
                     <geometry>
-                        <mesh filename="package://chassis_sub.SLDASM/meshes/chassis_link.STL" />
+                        <mesh filename="package://bot_description/meshes/body_link.STL" />
                     </geometry>
                     <material name="">
-                        <color rgba="0.5451 0.61569 0.85882 1" />
+                        <color rgba="0.792156862745098 0.819607843137255 0.933333333333333 1" />
                     </material>
                 </visual>
@@ -23,5 +23,5 @@
                     <origin xyz="0 0 0" rpy="0 0 0" />
                     <geometry>
-                        <mesh filename="package://bot_description/meshes/chassis_link.STL" />
+                        <mesh filename="package://bot_description/meshes/body_link.STL" />
                     </geometry>
                 </collision>

File: ros2_ws/src/bot_description/urdf/limb.urdf.xacro (robot description, xacro)
@@ -9,8 +9,8 @@
         <link name="${prefix}shoulder_link">
             <inertial>
-                <origin xyz="0.00123926352361432 0.00335245027216135 0.020963936804564" rpy="0 0 0" />
-                <mass value="0.0703942212311305" />
-                <inertia ixx="2.76576288052366E-05" ixy="-1.39471839648609E-07" ixz="-2.88488463706858E-07"
-                         iyy="1.71370747114446E-05" iyz="-6.19746545161347E-08" izz="2.60685249875832E-05" />
+                <origin xyz="0.00156778084450622 0.00023011490355522 0.0188653348885318" rpy="0 0 0" />
+                <mass value="0.0668523982562037" />
+                <inertia ixx="2.59076494418216E-05" ixy="-7.12609209313921E-08" ixz="-3.38158087429427E-07"
+                         iyy="1.53510229543711E-05" iyz="-2.56253037144619E-08" izz="2.5742400586002E-05" />
             </inertial>
             <visual>
@@ -32,8 +32,8 @@
         <link name="${prefix}femur_link">
             <inertial>
-                <origin xyz="0.0219749723740116 1.10674379296058E-05 0.0317318417810033" rpy="0 0 0" />
-                <mass value="0.0578650759594537" />
-                <inertia ixx="7.21606846133888E-06" ixy="-2.43047276138592E-09" ixz="-8.71808476080296E-07"
-                         iyy="3.86361231869082E-05" iyz="-9.13958901614113E-10" izz="3.73315278091681E-05" />
+                <origin xyz="0.0273832027524642 -0.00204211137254596 0.0280691114483194" rpy="0 0 0" />
+                <mass value="0.0660310589468222" />
+                <inertia ixx="1.26372174256358E-05" ixy="-2.79354262209908E-09" ixz="-1.19244684545251E-07"
+                         iyy="4.86450881022467E-05" iyz="-4.57382172664923E-07" izz="4.44007499741371E-05" />
             </inertial>
             <visual>
@@ -43,5 +43,5 @@
                 </geometry>
                 <material name="">
-                    <color rgba="0.96078431372549 0.96078431372549 0.964705882352941 1" />
+                    <color rgba="0.545098039215686 0.615686274509804 0.858823529411765 1" />
                 </material>
             </visual>
@@ -55,8 +55,8 @@
         <link name="${prefix}tibia_link">
             <inertial>
-                <origin xyz="0.031878867699759 5.86889321863016E-11 1.81508030133726E-08" rpy="0 0 0" />
-                <mass value="0.0109091234821787" />
-                <inertia ixx="1.95526217620308E-07" ixy="1.4570117043835E-11" ixz="1.85497777908555E-11"
-                         iyy="1.01874475115624E-05" iyz="-4.19910780669847E-12" izz="1.01972686884836E-05" />
+                <origin xyz="0.0288498831722294 -2.12695301857191E-07 -1.69859593279753E-07" rpy="0 0 0" />
+                <mass value="0.012227756457296" />
+                <inertia ixx="2.38144473002711E-07" ixy="4.86549409070109E-11" ixz="2.95033296846384E-11"
+                         iyy="8.84429570059483E-06" iyz="-1.13332312820773E-11" izz="8.85815361606418E-06" />
             </inertial>
             <visual>
@@ -77,5 +77,5 @@
         </link>
         <joint name="${prefix}hfe_joint" type="revolute">
-            <origin xyz="0.02088 0 0.0165" rpy="1.5708 ${0.0 if mult > 0 else 3.1416} 1.5708"/>
+            <origin xyz="0.0198 -0.0124999999999998 0.0215" rpy="-1.5707963267949 0.0843795007429648 -1.5707963267949"/>
             <parent link="${prefix}shoulder_link"/>
             <child link="${prefix}femur_link"/>
@@ -87,5 +87,5 @@
         </joint>
         <joint name="${prefix}kfe_joint" type="revolute">
-            <origin xyz="0.046 0 0.0106" rpy="0 0 0"/>
+            <origin xyz="0.096057287853238 0 0.0200000000000001" rpy="-3.14159265358979 0 -0.0843795007429648"/>
             <parent link="${prefix}femur_link"/>
             <child link="${prefix}tibia_link"/>

File: ros2_ws/src/bot_description/urdf/robot.urdf.xacro (robot description, xacro)
@@ -5,10 +5,11 @@
     <!-- Hardware args -->
     <xacro:arg name="hardware_plugin" default="mock_components/GenericSystem"/>
-    <!-- Common leg placement/orientation values -->
-    <xacro:property name="leg_x" value="-0.04991"/>
-    <xacro:property name="leg_y" value="-0.0056409"/>
-    <xacro:property name="leg_z" value="-0.066876"/>
-    <xacro:property name="leg_pitch" value="1.5708"/>
-    <xacro:property name="leg_roll_flip" value="3.1416"/>
+    <!-- Common leg placement/orientation values (from chassis_sub.SLDASM export, single reference limb) -->
+    <xacro:property name="leg_x" value="-0.0828"/>
+    <xacro:property name="leg_y" value="-0.056"/>
+    <xacro:property name="leg_z" value="0.0285"/>
+    <xacro:property name="leg_roll" value="1.5708"/>
+    <xacro:property name="leg_pitch" value="0"/>
+    <xacro:property name="leg_yaw" value="-1.5708"/>
     <!-- Import macros from other files -->
     <xacro:include filename="$(find bot_description)/urdf/body.urdf.xacro"/>
@@ -18,11 +19,9 @@
     <!-- Call macros -->
     <xacro:body/>
-    <xacro:limb prefix="fr" x="${leg_x}" y="${leg_y}" z="${-leg_z}" r="0" p="${leg_pitch}" yw="0" mult="1"/>
-    <xacro:limb prefix="fl" x="${leg_x}" y="${leg_y}" z="${leg_z}" r="${leg_roll_flip}" p="${-leg_pitch}" yw="0"
-                mult="-1"/>
-    <xacro:limb prefix="br" x="${-leg_x}" y="${leg_y}" z="${-leg_z}" r="${leg_roll_flip}" p="${leg_pitch}" yw="0"
-                mult="-1"/>
-    <xacro:limb prefix="bl" x="${-leg_x}" y="${leg_y}" z="${leg_z}" r="0" p="${-leg_pitch}" yw="0" mult="1"/>
-    <!-- macros specific to sim/hardware modes -->
+    <xacro:limb prefix="fl" x="${leg_x}" y="${leg_y}" z="${leg_z}" r="${leg_roll}" p="${leg_pitch}" yw="${leg_yaw}" mult="1"/>
+    <xacro:limb prefix="br" x="${-leg_x}" y="${-leg_y}" z="${leg_z}" r="${leg_roll}" p="${leg_pitch}" yw="${-leg_yaw}" mult="-1"/>
+    <!--<xacro:limb prefix="fr" .../>-->
+    <!--<xacro:limb prefix="bl" .../>-->
+     macros specific to sim/hardware modes
     <xacro:if value="$(arg sim)">
         <xacro:ros2_control name="GazeboSystem" hardware_plugin="gz_ros2_control/GazeboSimSystem"/>
