Commit message: feat(urdf): correctly position hfe and kfe joints

File: ros2_ws/src/bot_description/urdf/limb.urdf.xacro (robot description, xacro)
@@ -2,127 +2,127 @@
 <robot xmlns:xacro="http://www.ros.org/wiki/xacro" name="limb">
     <xacro:macro name="limb" params="prefix">
-    <!-- Links -->
-    <link name="${prefix}shoulder_link">
-        <inertial>
-            <origin xyz="0.018766 0.016329 0.0079907" rpy="0 0 0"/>
-            <mass value="0.01481"/>
-            <inertia ixx="1.3996E-06" ixy="-1.6833E-08" ixz="-7.906E-10" iyy="1.8819E-06" iyz="-3.0123E-10"
-                     izz="2.5913E-06"/>
-        </inertial>
-        <visual>
-            <origin xyz="0 0 0" rpy="0 0 0"/>
-            <geometry>
-                <mesh filename="package://bot_description/meshes/haa_horn.STL" scale="1 1 1"/>
-            </geometry>
-        </visual>
-        <visual>
-            <origin xyz="0 0 0" rpy="0 0 0"/>
-            <geometry>
-                <mesh filename="package://bot_description/meshes/shoulder_casing.STL" scale="1 1 1"/>
-            </geometry>
-        </visual>
-        <visual>
-            <origin xyz="0 0 0" rpy="0 0 0"/>
-            <geometry>
-                <mesh filename="package://bot_description/meshes/hfe_servo.STL" scale="1 1 1"/>
-            </geometry>
-        </visual>
-        <collision>
-            <origin xyz="0 0 0" rpy="0 0 0"/>
-            <geometry>
-                <mesh filename="package://bot_description/meshes/haa_horn.STL" scale="1 1 1"/>
-            </geometry>
-        </collision>
-        <collision>
-            <origin xyz="0 0 0" rpy="0 0 0"/>
-            <geometry>
-                <mesh filename="package://bot_description/meshes/shoulder_casing.STL" scale="1 1 1"/>
-            </geometry>
-        </collision>
-        <collision>
-            <origin xyz="0 0 0" rpy="0 0 0"/>
-            <geometry>
-                <mesh filename="package://bot_description/meshes/hfe_servo.STL" scale="1 1 1"/>
-            </geometry>
-        </collision>
-    </link>
-<!--    <link name="femur_link">-->
-<!--        <inertial>-->
-<!--            <origin xyz="0.012387 -0.00071898 0.017314" rpy="0 0 0"/>-->
-<!--            <mass value="0.015915"/>-->
-<!--            <inertia ixx="9.3139E-07" ixy="-7.9194E-10" ixz="-9.4792E-08" iyy="3.7356E-06" iyz="1.3143E-09"-->
-<!--                     izz="3.3585E-06"/>-->
-<!--        </inertial>-->
-<!--        <visual>-->
-<!--            <origin xyz="0 0 0" rpy="0 0 0"/>-->
-<!--            <geometry>-->
-<!--                <mesh filename="package://bot_description/meshes/hfe_horn.STL" scale="1 1 1"/>-->
-<!--            </geometry>-->
-<!--        </visual>-->
-<!--        <visual>-->
-<!--            <origin xyz="0 0 0" rpy="0 0 0"/>-->
-<!--            <geometry>-->
-<!--                <mesh filename="package://bot_description/meshes/femur.STL" scale="1 1 1"/>-->
-<!--            </geometry>-->
-<!--        </visual>-->
-<!--        <visual>-->
-<!--            <origin xyz="0 0 0" rpy="0 0 0"/>-->
-<!--            <geometry>-->
-<!--                <mesh filename="package://bot_description/meshes/kfe_servo.STL" scale="1 1 1"/>-->
-<!--            </geometry>-->
-<!--        </visual>-->
-<!--        <collision>-->
-<!--            <origin xyz="0 0 0" rpy="0 0 0"/>-->
-<!--            <geometry>-->
-<!--                <mesh filename="package://bot_description/meshes/hfe_horn.STL" scale="1 1 1"/>-->
-<!--            </geometry>-->
-<!--        </collision>-->
-<!--        <collision>-->
-<!--            <origin xyz="0 0 0" rpy="0 0 0"/>-->
-<!--            <geometry>-->
-<!--                <mesh filename="package://bot_description/meshes/femur.STL" scale="1 1 1"/>-->
-<!--            </geometry>-->
-<!--        </collision>-->
-<!--        <collision>-->
-<!--            <origin xyz="0 0 0" rpy="0 0 0"/>-->
-<!--            <geometry>-->
-<!--                <mesh filename="package://bot_description/meshes/kfe_servo.STL" scale="1 1 1"/>-->
-<!--            </geometry>-->
-<!--        </collision>-->
-<!--    </link>-->
-<!--    <link name="tibia_link">-->
-<!--        <inertial>-->
-<!--            <origin xyz="0.0019117 0.036934 -0.0058072" rpy="0 0 0"/>-->
-<!--            <mass value="0.052333"/>-->
-<!--            <inertia ixx="3.6178E-05" ixy="3.873E-06" ixz="-6.0786E-07" iyy="2.0314E-05" iyz="6.2224E-06"-->
-<!--                     izz="2.4513E-05"/>-->
-<!--        </inertial>-->
-<!--        <visual>-->
-<!--            <origin xyz="0 0 0" rpy="0 0 0"/>-->
-<!--            <geometry>-->
-<!--                <mesh filename="package://bot_description/meshes/tibia.STL" scale="1 1 1"/>-->
-<!--            </geometry>-->
-<!--        </visual>-->
-<!--        <collision>-->
-<!--            <origin xyz="0 0 0" rpy="0 0 0"/>-->
-<!--            <geometry>-->
-<!--                <mesh filename="package://bot_description/meshes/tibia.STL" scale="1 1 1"/>-->
-<!--            </geometry>-->
-<!--        </collision>-->
-<!--    </link>-->
-<!--    <joint name="hfe_joint" type="revolute">-->
-<!--        <origin xyz="0.023 -1.008 0.0295" rpy="3.14 -1.5708 0 "/>-->
-<!--        <parent link="shoulder_link"/>-->
-<!--        <child link="femur_link"/>-->
-<!--        <axis xyz="0 0 -1"/>-->
-<!--        <limit lower="0" upper="0" effort="0" velocity="0"/>-->
-<!--    </joint>-->
-<!--    <joint name="kfe_joint" type="revolute">-->
-<!--        <origin xyz="0.046 0 0.0106" rpy="0 0 1.5708"/>-->
-<!--        <parent link="femur_link"/>-->
-<!--        <child link="tibia_link"/>-->
-<!--        <axis xyz="0 0 -1"/>-->
-<!--        <limit lower="0" upper="0" effort="50" velocity="50"/>-->
-<!--    </joint>-->
+        <!-- Links -->
+        <link name="${prefix}shoulder_link">
+            <inertial>
+                <origin xyz="0.018766 0.016329 0.0079907" rpy="0 0 0"/>
+                <mass value="0.01481"/>
+                <inertia ixx="1.3996E-06" ixy="-1.6833E-08" ixz="-7.906E-10" iyy="1.8819E-06" iyz="-3.0123E-10"
+                         izz="2.5913E-06"/>
+            </inertial>
+            <visual>
+                <origin xyz="0 0 0" rpy="0 0 0"/>
+                <geometry>
+                    <mesh filename="package://bot_description/meshes/haa_horn.STL" scale="1 1 1"/>
+                </geometry>
+            </visual>
+            <visual>
+                <origin xyz="0 0 0" rpy="0 0 0"/>
+                <geometry>
+                    <mesh filename="package://bot_description/meshes/shoulder_casing.STL" scale="1 1 1"/>
+                </geometry>
+            </visual>
+            <visual>
+                <origin xyz="0 0 0" rpy="0 0 0"/>
+                <geometry>
+                    <mesh filename="package://bot_description/meshes/hfe_servo.STL" scale="1 1 1"/>
+                </geometry>
+            </visual>
+            <collision>
+                <origin xyz="0 0 0" rpy="0 0 0"/>
+                <geometry>
+                    <mesh filename="package://bot_description/meshes/haa_horn.STL" scale="1 1 1"/>
+                </geometry>
+            </collision>
+            <collision>
+                <origin xyz="0 0 0" rpy="0 0 0"/>
+                <geometry>
+                    <mesh filename="package://bot_description/meshes/shoulder_casing.STL" scale="1 1 1"/>
+                </geometry>
+            </collision>
+            <collision>
+                <origin xyz="0 0 0" rpy="0 0 0"/>
+                <geometry>
+                    <mesh filename="package://bot_description/meshes/hfe_servo.STL" scale="1 1 1"/>
+                </geometry>
+            </collision>
+        </link>
+        <link name="${prefix}femur_link">
+            <inertial>
+                <origin xyz="0.012387 -0.00071898 0.017314" rpy="0 0 0"/>
+                <mass value="0.015915"/>
+                <inertia ixx="9.3139E-07" ixy="-7.9194E-10" ixz="-9.4792E-08" iyy="3.7356E-06" iyz="1.3143E-09"
+                         izz="3.3585E-06"/>
+            </inertial>
+            <visual>
+                <origin xyz="0 0 0" rpy="0 0 0"/>
+                <geometry>
+                    <mesh filename="package://bot_description/meshes/hfe_horn.STL" scale="1 1 1"/>
+                </geometry>
+            </visual>
+            <visual>
+                <origin xyz="0 0 0" rpy="0 0 0"/>
+                <geometry>
+                    <mesh filename="package://bot_description/meshes/femur.STL" scale="1 1 1"/>
+                </geometry>
+            </visual>
+            <visual>
+                <origin xyz="0 0 0" rpy="0 0 0"/>
+                <geometry>
+                    <mesh filename="package://bot_description/meshes/kfe_servo.STL" scale="1 1 1"/>
+                </geometry>
+            </visual>
+            <collision>
+                <origin xyz="0 0 0" rpy="0 0 0"/>
+                <geometry>
+                    <mesh filename="package://bot_description/meshes/hfe_horn.STL" scale="1 1 1"/>
+                </geometry>
+            </collision>
+            <collision>
+                <origin xyz="0 0 0" rpy="0 0 0"/>
+                <geometry>
+                    <mesh filename="package://bot_description/meshes/femur.STL" scale="1 1 1"/>
+                </geometry>
+            </collision>
+            <collision>
+                <origin xyz="0 0 0" rpy="0 0 0"/>
+                <geometry>
+                    <mesh filename="package://bot_description/meshes/kfe_servo.STL" scale="1 1 1"/>
+                </geometry>
+            </collision>
+        </link>
+        <link name="${prefix}tibia_link">
+            <inertial>
+                <origin xyz="0.0019117 0.036934 -0.0058072" rpy="0 0 0"/>
+                <mass value="0.052333"/>
+                <inertia ixx="3.6178E-05" ixy="3.873E-06" ixz="-6.0786E-07" iyy="2.0314E-05" iyz="6.2224E-06"
+                         izz="2.4513E-05"/>
+            </inertial>
+            <visual>
+                <origin xyz="0 0 0" rpy="0 0 0"/>
+                <geometry>
+                    <mesh filename="package://bot_description/meshes/tibia.STL" scale="1 1 1"/>
+                </geometry>
+            </visual>
+            <collision>
+                <origin xyz="0 0 0" rpy="0 0 0"/>
+                <geometry>
+                    <mesh filename="package://bot_description/meshes/tibia.STL" scale="1 1 1"/>
+                </geometry>
+            </collision>
+        </link>
+        <joint name="${prefix}hfe_joint" type="revolute">
+            <origin xyz="0.02088 0 0.0165" rpy="3.1416 -1.5708 0 "/>
+            <parent link="${prefix}shoulder_link"/>
+            <child link="${prefix}femur_link"/>
+            <axis xyz="0 0 -1"/>
+            <limit lower="0" upper="0" effort="0" velocity="0"/>
+        </joint>
+        <joint name="${prefix}kfe_joint" type="revolute">
+            <origin xyz="0.046 0 0.0106" rpy="0 0 -1.5708"/>
+            <parent link="${prefix}femur_link"/>
+            <child link="${prefix}tibia_link"/>
+            <axis xyz="0 0 -1"/>
+            <limit lower="0" upper="0" effort="50" velocity="50"/>
+        </joint>
     </xacro:macro>
 </robot>

Commit message: feat(ros/bot_description): correctly connect the inverted limbs (fl and br)

File: ros2_ws/src/bot_description/urdf/limb.urdf.xacro (robot description, xacro)
@@ -1,5 +1,5 @@
 <?xml version="1.0" encoding="utf-8"?>
 <robot xmlns:xacro="http://www.ros.org/wiki/xacro" name="limb">
-    <xacro:macro name="limb" params="prefix">
+    <xacro:macro name="limb" params="prefix mult">
         <!-- Links -->
         <link name="${prefix}shoulder_link">
@@ -112,5 +112,5 @@
         </link>
         <joint name="${prefix}hfe_joint" type="revolute">
-            <origin xyz="0.02088 0 0.0165" rpy="3.1416 -1.5708 0 "/>
+            <origin xyz="0.02088 0 0.0165" rpy="${mult * 3.1416} -1.5708 0 "/>
             <parent link="${prefix}shoulder_link"/>
             <child link="${prefix}femur_link"/>
@@ -119,5 +119,5 @@
         </joint>
         <joint name="${prefix}kfe_joint" type="revolute">
-            <origin xyz="0.046 0 0.0106" rpy="0 0 -1.5708"/>
+            <origin xyz="0.046 0 0.0106" rpy="0 0 ${mult * -1.5708}"/>
             <parent link="${prefix}femur_link"/>
             <child link="${prefix}tibia_link"/>

File: ros2_ws/src/bot_description/urdf/robot.urdf.xacro (robot description, xacro)
@@ -5,6 +5,6 @@
     <xacro:include filename="$(find bot_description)/urdf/limb.urdf.xacro"/>
     <!-- Macro that adds a limb and joints it to body -->
-    <xacro:macro name="add_limb" params="prefix x y z r p yw">
-        <xacro:limb prefix="${prefix}_"/>
+    <xacro:macro name="add_limb" params="prefix x y z r p yw mult">
+        <xacro:limb prefix="${prefix}_" mult="${mult}"/>
         <joint name="${prefix}_haa_joint" type="revolute">
             <parent link="body_link"/>
@@ -16,7 +16,7 @@
     </xacro:macro>
     <xacro:body/>
-    <xacro:add_limb prefix="fl" x="0.0765"  y="-0.009" z="-0.0338" r="0" p="1.5708"  yw="0"/>
-<!--    <xacro:add_limb prefix="fr" x="0.0765"  y="-0.009" z="0.0338"  r="0" p="1.5708"  yw="0"/>-->
-<!--    <xacro:add_limb prefix="bl" x="-0.0765" y="-0.009" z="-0.0338" r="0" p="-1.5708" yw="0"/>-->
-    <xacro:add_limb prefix="br" x="-0.0765" y="-0.009" z="0.0338"  r="0" p="-1.5708" yw="0"/>
+    <xacro:add_limb prefix="fr" x="0.0765" y="-0.009" z="-0.0338" r="0" p="1.5708" yw="0" mult="1"/>
+    <xacro:add_limb prefix="fl" x="0.0765"  y="-0.009" z="0.0338"  r="3.1416" p="-1.5708"  yw="0" mult="-1"/>
+    <xacro:add_limb prefix="br" x="-0.0765" y="-0.009" z="-0.0338" r="3.1416" p="1.5708" yw="0" mult="-1"/>
+    <xacro:add_limb prefix="bl" x="-0.0765" y="-0.009" z="0.0338" r="0" p="-1.5708" yw="0" mult="1"/>
 </robot>

Commit message: chore(ros/bot_description): use xacro props for constant

File: ros2_ws/src/bot_description/urdf/limb.urdf.xacro (robot description, xacro)
@@ -1,4 +1,8 @@
 <?xml version="1.0" encoding="utf-8"?>
 <robot xmlns:xacro="http://www.ros.org/wiki/xacro" name="limb">
+    <!-- Joint limits loaded from YAML -->
+    <xacro:property name="limits"
+                    value="${xacro.load_yaml('$(find bot_description)/config/joint_limits.yaml')}"/>
+    <!-- Limb macro definition -->
     <xacro:macro name="limb" params="prefix mult">
         <!-- Links -->
@@ -112,9 +116,12 @@
         </link>
         <joint name="${prefix}hfe_joint" type="revolute">
-            <origin xyz="0.02088 0 0.0165" rpy="${mult * 3.1416} -1.5708 0 "/>
+            <origin xyz="0.02088 0 0.0165" rpy="3.1416 -1.5708 0 "/>
             <parent link="${prefix}shoulder_link"/>
             <child link="${prefix}femur_link"/>
             <axis xyz="0 0 -1"/>
-            <limit lower="0" upper="0" effort="0" velocity="0"/>
+            <limit lower="${limits['hfe']['lower']}"
+                   upper="${limits['hfe']['upper']}"
+                   effort="${limits['hfe']['effort']}"
+                   velocity="${limits['hfe']['velocity']}"/>
         </joint>
         <joint name="${prefix}kfe_joint" type="revolute">
@@ -123,5 +130,8 @@
             <child link="${prefix}tibia_link"/>
             <axis xyz="0 0 -1"/>
-            <limit lower="0" upper="0" effort="50" velocity="50"/>
+            <limit lower="${limits['kfe']['lower']}"
+                   upper="${limits['kfe']['upper']}"
+                   effort="${limits['kfe']['effort']}"
+                   velocity="${limits['kfe']['velocity']}"/>
         </joint>
     </xacro:macro>

File: ros2_ws/src/bot_description/urdf/robot.urdf.xacro (robot description, xacro)
@@ -1,4 +1,13 @@
 <?xml version="1.0"?>
 <robot xmlns:xacro="http://www.ros.org/wiki/xacro" name="quad_quad_bot">
+    <!-- Common leg placement/orientation constants -->
+    <xacro:property name="leg_x" value="0.0765"/>
+    <xacro:property name="leg_y" value="-0.009"/>
+    <xacro:property name="leg_z" value="0.0338"/>
+    <xacro:property name="leg_pitch" value="1.5708"/>
+    <xacro:property name="leg_roll_flip" value="3.1416"/>
+    <!-- Joint limits loaded from YAML -->
+    <xacro:property name="limits"
+                    value="${xacro.load_yaml('$(find bot_description)/config/joint_limits.yaml')}"/>
     <!-- Parts from other files -->
     <xacro:include filename="$(find bot_description)/urdf/body.urdf.xacro"/>
@@ -12,11 +21,17 @@
             <origin xyz="${x} ${y} ${z}" rpy="${r} ${p} ${yw}"/>
             <axis xyz="0 0 1"/>
-            <limit lower="-3.14" upper="3.14" effort="1000" velocity="5"/>
+            <limit lower="${limits['haa']['lower']}"
+                   upper="${limits['haa']['upper']}"
+                   effort="${limits['haa']['effort']}"
+                   velocity="${limits['haa']['velocity']}"/>
         </joint>
     </xacro:macro>
+    <!-- Call macros -->
     <xacro:body/>
-    <xacro:add_limb prefix="fr" x="0.0765" y="-0.009" z="-0.0338" r="0" p="1.5708" yw="0" mult="1"/>
-    <xacro:add_limb prefix="fl" x="0.0765"  y="-0.009" z="0.0338"  r="3.1416" p="-1.5708"  yw="0" mult="-1"/>
-    <xacro:add_limb prefix="br" x="-0.0765" y="-0.009" z="-0.0338" r="3.1416" p="1.5708" yw="0" mult="-1"/>
-    <xacro:add_limb prefix="bl" x="-0.0765" y="-0.009" z="0.0338" r="0" p="-1.5708" yw="0" mult="1"/>
+    <xacro:add_limb prefix="fr" x="${leg_x}" y="${leg_y}" z="${-leg_z}" r="0" p="${leg_pitch}" yw="0" mult="1"/>
+    <xacro:add_limb prefix="fl" x="${leg_x}" y="${leg_y}" z="${leg_z}" r="${leg_roll_flip}" p="${-leg_pitch}" yw="0"
+                    mult="-1"/>
+    <xacro:add_limb prefix="br" x="${-leg_x}" y="${leg_y}" z="${-leg_z}" r="${leg_roll_flip}" p="${leg_pitch}" yw="0"
+                    mult="-1"/>
+    <xacro:add_limb prefix="bl" x="${-leg_x}" y="${leg_y}" z="${leg_z}" r="0" p="${-leg_pitch}" yw="0" mult="1"/>
 </robot>

Commit message: refactor(ros/robot_description): encapsulate limb assembly in limb macro and remove robot add_limb

File: ros2_ws/src/bot_description/urdf/limb.urdf.xacro (robot description, xacro)
@@ -4,6 +4,6 @@
     <xacro:property name="limits"
                     value="${xacro.load_yaml('$(find bot_description)/config/joint_limits.yaml')}"/>
-    <!-- Limb macro definition -->
-    <xacro:macro name="limb" params="prefix mult">
+    <!-- Internal limb geometry + internal joints (hfe/kfe). -->
+    <xacro:macro name="_limb_core" params="prefix mult">
         <!-- Links -->
         <link name="${prefix}shoulder_link">
@@ -136,3 +136,17 @@
         </joint>
     </xacro:macro>
+    <!-- Public limb macro: owns full attachment to body, hiding internal limb construction. -->
+    <xacro:macro name="limb" params="prefix x y z r p yw mult parent_link:=body_link">
+        <xacro:_limb_core prefix="${prefix}_" mult="${mult}"/>
+        <joint name="${prefix}_haa_joint" type="revolute">
+            <parent link="${parent_link}"/>
+            <child link="${prefix}_shoulder_link"/>
+            <origin xyz="${x} ${y} ${z}" rpy="${r} ${p} ${yw}"/>
+            <axis xyz="0 0 1"/>
+            <limit lower="${limits['haa']['lower']}"
+                   upper="${limits['haa']['upper']}"
+                   effort="${limits['haa']['effort']}"
+                   velocity="${limits['haa']['velocity']}"/>
+        </joint>
+    </xacro:macro>
 </robot>

File: ros2_ws/src/bot_description/urdf/robot.urdf.xacro (robot description, xacro)
@@ -7,31 +7,14 @@
     <xacro:property name="leg_pitch" value="1.5708"/>
     <xacro:property name="leg_roll_flip" value="3.1416"/>
-    <!-- Joint limits loaded from YAML -->
-    <xacro:property name="limits"
-                    value="${xacro.load_yaml('$(find bot_description)/config/joint_limits.yaml')}"/>
     <!-- Parts from other files -->
     <xacro:include filename="$(find bot_description)/urdf/body.urdf.xacro"/>
     <xacro:include filename="$(find bot_description)/urdf/limb.urdf.xacro"/>
-    <!-- Macro that adds a limb and joints it to body -->
-    <xacro:macro name="add_limb" params="prefix x y z r p yw mult">
-        <xacro:limb prefix="${prefix}_" mult="${mult}"/>
-        <joint name="${prefix}_haa_joint" type="revolute">
-            <parent link="body_link"/>
-            <child link="${prefix}_shoulder_link"/>
-            <origin xyz="${x} ${y} ${z}" rpy="${r} ${p} ${yw}"/>
-            <axis xyz="0 0 1"/>
-            <limit lower="${limits['haa']['lower']}"
-                   upper="${limits['haa']['upper']}"
-                   effort="${limits['haa']['effort']}"
-                   velocity="${limits['haa']['velocity']}"/>
-        </joint>
-    </xacro:macro>
     <!-- Call macros -->
     <xacro:body/>
-    <xacro:add_limb prefix="fr" x="${leg_x}" y="${leg_y}" z="${-leg_z}" r="0" p="${leg_pitch}" yw="0" mult="1"/>
-    <xacro:add_limb prefix="fl" x="${leg_x}" y="${leg_y}" z="${leg_z}" r="${leg_roll_flip}" p="${-leg_pitch}" yw="0"
-                    mult="-1"/>
-    <xacro:add_limb prefix="br" x="${-leg_x}" y="${leg_y}" z="${-leg_z}" r="${leg_roll_flip}" p="${leg_pitch}" yw="0"
-                    mult="-1"/>
-    <xacro:add_limb prefix="bl" x="${-leg_x}" y="${leg_y}" z="${leg_z}" r="0" p="${-leg_pitch}" yw="0" mult="1"/>
+    <xacro:limb prefix="fr" x="${leg_x}" y="${leg_y}" z="${-leg_z}" r="0" p="${leg_pitch}" yw="0" mult="1"/>
+    <xacro:limb prefix="fl" x="${leg_x}" y="${leg_y}" z="${leg_z}" r="${leg_roll_flip}" p="${-leg_pitch}" yw="0"
+                mult="-1"/>
+    <xacro:limb prefix="br" x="${-leg_x}" y="${leg_y}" z="${-leg_z}" r="${leg_roll_flip}" p="${leg_pitch}" yw="0"
+                mult="-1"/>
+    <xacro:limb prefix="bl" x="${-leg_x}" y="${leg_y}" z="${leg_z}" r="0" p="${-leg_pitch}" yw="0" mult="1"/>
 </robot>

Commit message: refactor(urdf): redefine limb joint origins so zero angles match I-pose

File: ros2_ws/src/bot_description/urdf/limb.urdf.xacro (robot description, xacro)
@@ -116,5 +116,5 @@
         </link>
         <joint name="${prefix}hfe_joint" type="revolute">
-            <origin xyz="0.02088 0 0.0165" rpy="3.1416 -1.5708 0 "/>
+            <origin xyz="0.02088 0 0.0165" rpy="1.5708 ${0.0 if mult > 0 else 3.1416} 1.5708"/>
             <parent link="${prefix}shoulder_link"/>
             <child link="${prefix}femur_link"/>
@@ -126,5 +126,5 @@
         </joint>
         <joint name="${prefix}kfe_joint" type="revolute">
-            <origin xyz="0.046 0 0.0106" rpy="0 0 ${mult * -1.5708}"/>
+            <origin xyz="0.046 0 0.0106" rpy="0 0 0"/>
             <parent link="${prefix}femur_link"/>
             <child link="${prefix}tibia_link"/>
