Commit message: refactor(urdf): normalize limb joint axis directions across all legs

File: ros2_ws/src/bot_description/urdf/limb.urdf.xacro (robot description, xacro)
@@ -119,5 +119,5 @@
             <parent link="${prefix}shoulder_link"/>
             <child link="${prefix}femur_link"/>
-            <axis xyz="0 0 -1"/>
+            <axis xyz="0 0 ${mult * 1}"/>
             <limit lower="${limits['hfe']['lower']}"
                    upper="${limits['hfe']['upper']}"
@@ -129,5 +129,5 @@
             <parent link="${prefix}femur_link"/>
             <child link="${prefix}tibia_link"/>
-            <axis xyz="0 0 -1"/>
+            <axis xyz="0 0 ${mult * -1}"/>
             <limit lower="${limits['kfe']['lower']}"
                    upper="${limits['kfe']['upper']}"
@@ -143,5 +143,5 @@
             <child link="${prefix}_shoulder_link"/>
             <origin xyz="${x} ${y} ${z}" rpy="${r} ${p} ${yw}"/>
-            <axis xyz="0 0 1"/>
+            <axis xyz="0 0 ${mult * -1}"/>
             <limit lower="${limits['haa']['lower']}"
                    upper="${limits['haa']['upper']}"

Commit message: feat(urdf): implement updates into xacro

File: ros2_ws/src/bot_description/urdf/limb.urdf.xacro (robot description, xacro)
@@ -5,17 +5,22 @@
                     value="${xacro.load_yaml('$(find bot_description)/config/joint_limits.yaml')}"/>
     <!-- Internal limb geometry + internal joints (hfe/kfe). -->
-    <xacro:macro name="_limb_core" params="prefix mult">
+    <xacro:macro name="_limb_core" params="prefix inverted_shoulder">
         <!-- Links -->
         <link name="${prefix}shoulder_link">
             <inertial>
-                <origin xyz="0.00156778084450622 0.00023011490355522 0.0188653348885318" rpy="0 0 0" />
-                <mass value="0.0668523982562037" />
-                <inertia ixx="2.59076494418216E-05" ixy="-7.12609209313921E-08" ixz="-3.38158087429427E-07"
-                         iyy="1.53510229543711E-05" iyz="-2.56253037144619E-08" izz="2.5742400586002E-05" />
+                <origin xyz="0.00189283967211911 -0.00149022104022392 0.0209651260942884" rpy="0 0 0" />
+                <mass value="0.0772984767866564" />
+                <inertia ixx="2.74184679471754E-05" ixy="-7.12325596084157E-08" ixz="1.19608410119039E-07"
+                         iyy="2.07506136746851E-05" iyz="-2.5629423337733E-08" izz="3.03168099471715E-05" />
             </inertial>
             <visual>
                 <origin xyz="0 0 0" rpy="0 0 0"/>
                 <geometry>
-                    <mesh filename="package://bot_description/meshes/shoulder_link.STL" />
+                    <xacro:if value="${inverted_shoulder}">
+                        <mesh filename="package://bot_description/meshes/inverted_shoulder_link.STL" scale="0.001 0.001 0.001"/>
+                    </xacro:if>
+                    <xacro:unless value="${inverted_shoulder}">
+                        <mesh filename="package://bot_description/meshes/shoulder_link.STL" scale="1 1 1" />
+                    </xacro:unless>
                 </geometry>
                 <material name="">
@@ -26,5 +31,10 @@
                 <origin xyz="0 0 0" rpy="0 0 0"/>
                 <geometry>
-                    <mesh filename="package://bot_description/meshes/shoulder_link.STL" scale="1 1 1"/>
+                    <xacro:if value="${inverted_shoulder}">
+                        <mesh filename="package://bot_description/meshes/inverted_shoulder_link.STL" scale="0.001 0.001 0.001"/>
+                    </xacro:if>
+                    <xacro:unless value="${inverted_shoulder}">
+                        <mesh filename="package://bot_description/meshes/shoulder_link.STL" scale="1 1 1"/>
+                    </xacro:unless>
                 </geometry>
             </collision>
@@ -32,8 +42,8 @@
         <link name="${prefix}femur_link">
             <inertial>
-                <origin xyz="0.0273832027524642 -0.00204211137254596 0.0280691114483194" rpy="0 0 0" />
-                <mass value="0.0660310589468222" />
-                <inertia ixx="1.26372174256358E-05" ixy="-2.79354262209908E-09" ixz="-1.19244684545251E-07"
-                         iyy="4.86450881022467E-05" iyz="-4.57382172664923E-07" izz="4.44007499741371E-05" />
+                <origin xyz="0.0323249229136636 -9.62316571824495E-07 0.0265797029719004" rpy="0 0 0" />
+                <mass value="0.0561441430721167" />
+                <inertia ixx="7.25316608559317E-06" ixy="-2.79260011877617E-09" ixz="-1.19212807601372E-07"
+                         iyy="4.40862958479968E-05" iyz="3.84318283091856E-10" izz="4.29206771962485E-05" />
             </inertial>
             <visual>
@@ -77,8 +87,8 @@
         </link>
         <joint name="${prefix}hfe_joint" type="revolute">
-            <origin xyz="0.0198 -0.0124999999999998 0.0215" rpy="-1.5707963267949 0.0843795007429648 -1.5707963267949"/>
+            <origin xyz="0.0298000000000001 -0.0124999999999999 0.0214999999999999" rpy="-1.5707963267949 0 -1.5707963267949"/>
             <parent link="${prefix}shoulder_link"/>
             <child link="${prefix}femur_link"/>
-            <axis xyz="0 0 ${mult * 1}"/>
+            <axis xyz="0 0 1"/>
             <limit lower="${limits['hfe']['lower']}"
                    upper="${limits['hfe']['upper']}"
@@ -87,8 +97,8 @@
         </joint>
         <joint name="${prefix}kfe_joint" type="revolute">
-            <origin xyz="0.096057287853238 0 0.0200000000000001" rpy="-3.14159265358979 0 -0.0843795007429648"/>
+            <origin xyz="0.0960572429044665 0 0.00999999999999993" rpy="-3.14159265358979 0 0"/>
             <parent link="${prefix}femur_link"/>
             <child link="${prefix}tibia_link"/>
-            <axis xyz="0 0 ${mult * -1}"/>
+            <axis xyz="0 0 -1"/>
             <limit lower="${limits['kfe']['lower']}"
                    upper="${limits['kfe']['upper']}"
@@ -98,11 +108,11 @@
     </xacro:macro>
     <!-- Public limb macro: owns full attachment to body, hiding internal limb construction. -->
-    <xacro:macro name="limb" params="prefix x y z r p yw mult parent_link:=body_link">
-        <xacro:_limb_core prefix="${prefix}_" mult="${mult}"/>
+    <xacro:macro name="limb" params="prefix x y z r p yw parent_link:=body_link inverted_shoulder">
+        <xacro:_limb_core prefix="${prefix}_" inverted_shoulder="${inverted_shoulder}"/>
         <joint name="${prefix}_haa_joint" type="revolute">
             <parent link="${parent_link}"/>
             <child link="${prefix}_shoulder_link"/>
             <origin xyz="${x} ${y} ${z}" rpy="${r} ${p} ${yw}"/>
-            <axis xyz="0 0 ${mult * -1}"/>
+            <axis xyz="0 0 -1"/>
             <limit lower="${limits['haa']['lower']}"
                    upper="${limits['haa']['upper']}"

File: ros2_ws/src/bot_description/urdf/robot.urdf.xacro (robot description, xacro)
@@ -19,8 +19,8 @@
     <!-- Call macros -->
     <xacro:body/>
-    <xacro:limb prefix="fl" x="${leg_x}" y="${leg_y}" z="${leg_z}" r="${leg_roll}" p="${leg_pitch}" yw="${leg_yaw}" mult="1"/>
-    <xacro:limb prefix="br" x="${-leg_x}" y="${-leg_y}" z="${leg_z}" r="${leg_roll}" p="${leg_pitch}" yw="${-leg_yaw}" mult="-1"/>
-    <!--<xacro:limb prefix="fr" .../>-->
-    <!--<xacro:limb prefix="bl" .../>-->
+    <xacro:limb prefix="fl" x="${leg_x}"  y="${leg_y}"  z="${leg_z}" r="${leg_roll}" p="${leg_pitch}" yw="${leg_yaw}"  inverted_shoulder="false"/>
+    <xacro:limb prefix="fr" x="${leg_x}"  y="${-leg_y}" z="${leg_z}" r="${leg_roll}" p="${leg_pitch}" yw="${-leg_yaw}" inverted_shoulder="true" />
+    <xacro:limb prefix="bl" x="${-leg_x}" y="${leg_y}"  z="${leg_z}" r="${leg_roll}" p="${leg_pitch}" yw="${leg_yaw}"  inverted_shoulder="true" />
+    <xacro:limb prefix="br" x="${-leg_x}" y="${-leg_y}" z="${leg_z}" r="${leg_roll}" p="${leg_pitch}" yw="${-leg_yaw}" inverted_shoulder="false"/>
      macros specific to sim/hardware modes
     <xacro:if value="$(arg sim)">

Commit message: fix(urdf): add appropriate inversion to femur joint on inverted shoudler side

File: ros2_ws/src/bot_description/urdf/limb.urdf.xacro (robot description, xacro)
@@ -87,5 +87,10 @@
         </link>
         <joint name="${prefix}hfe_joint" type="revolute">
-            <origin xyz="0.0298000000000001 -0.0124999999999999 0.0214999999999999" rpy="-1.5707963267949 0 -1.5707963267949"/>
+            <xacro:if value="${inverted_shoulder}">
+                <origin xyz="0.0298000000000001 -0.0124999999999999 -0.0214999999999999" rpy="-1.5707963267949 0 -1.5707963267949"/>
+            </xacro:if>
+            <xacro:unless value="${inverted_shoulder}">
+                <origin xyz="0.0298000000000001 -0.0124999999999999 0.0214999999999999" rpy="-1.5707963267949 0 -1.5707963267949"/>
+            </xacro:unless>
             <parent link="${prefix}shoulder_link"/>
             <child link="${prefix}femur_link"/>

Commit message: fix(urdf): add the missing end effector to xacro structure and remove redundant files

File: ros2_ws/src/bot_description/urdf/limb.urdf.xacro (robot description, xacro)
@@ -65,8 +65,8 @@
         <link name="${prefix}tibia_link">
             <inertial>
-                <origin xyz="0.0288498831722294 -2.12695301857191E-07 -1.69859593279753E-07" rpy="0 0 0" />
-                <mass value="0.012227756457296" />
-                <inertia ixx="2.38144473002711E-07" ixy="4.86549409070109E-11" ixz="2.95033296846384E-11"
-                         iyy="8.84429570059483E-06" iyz="-1.13332312820773E-11" izz="8.85815361606418E-06" />
+                <origin xyz="0.039043936151174 -1.78287788882986E-07 -1.41708728744472E-07" rpy="0 0 0" />
+                <mass value="0.0146532231932923" />
+                <inertia ixx="3.23322248550409E-07" ixy="4.86893510930891E-11" ixz="2.95568494794611E-11"
+                         iyy="8.9097637357867E-06" iyz="-1.13366884689962E-11" izz="8.92361996275972E-06" />
             </inertial>
             <visual>

Commit message: feat(urdf): perform needed inversions to follow angle direction conventions

File: ros2_ws/src/bot_description/urdf/limb.urdf.xacro (robot description, xacro)
@@ -5,5 +5,5 @@
                     value="${xacro.load_yaml('$(find bot_description)/config/joint_limits.yaml')}"/>
     <!-- Internal limb geometry + internal joints (hfe/kfe). -->
-    <xacro:macro name="_limb_core" params="prefix inverted_shoulder">
+    <xacro:macro name="_limb_core" params="prefix inverted_shoulder hfe_axis_mult kfe_axis_mult">
         <!-- Links -->
         <link name="${prefix}shoulder_link">
@@ -95,5 +95,5 @@
             <parent link="${prefix}shoulder_link"/>
             <child link="${prefix}femur_link"/>
-            <axis xyz="0 0 1"/>
+            <axis xyz="0 0 ${hfe_axis_mult * -1}"/>
             <limit lower="${limits['hfe']['lower']}"
                    upper="${limits['hfe']['upper']}"
@@ -105,5 +105,5 @@
             <parent link="${prefix}femur_link"/>
             <child link="${prefix}tibia_link"/>
-            <axis xyz="0 0 -1"/>
+            <axis xyz="0 0 ${kfe_axis_mult * 1}"/>
             <limit lower="${limits['kfe']['lower']}"
                    upper="${limits['kfe']['upper']}"
@@ -113,11 +113,11 @@
     </xacro:macro>
     <!-- Public limb macro: owns full attachment to body, hiding internal limb construction. -->
-    <xacro:macro name="limb" params="prefix x y z r p yw parent_link:=body_link inverted_shoulder">
-        <xacro:_limb_core prefix="${prefix}_" inverted_shoulder="${inverted_shoulder}"/>
+    <xacro:macro name="limb" params="prefix x y z r p yw parent_link:=body_link inverted_shoulder hfe_axis_mult kfe_axis_mult">
+        <xacro:_limb_core prefix="${prefix}_" inverted_shoulder="${inverted_shoulder}" hfe_axis_mult="${hfe_axis_mult}" kfe_axis_mult="${kfe_axis_mult}"/>
         <joint name="${prefix}_haa_joint" type="revolute">
             <parent link="${parent_link}"/>
             <child link="${prefix}_shoulder_link"/>
             <origin xyz="${x} ${y} ${z}" rpy="${r} ${p} ${yw}"/>
-            <axis xyz="0 0 -1"/>
+            <axis xyz="0 0 1"/>
             <limit lower="${limits['haa']['lower']}"
                    upper="${limits['haa']['upper']}"

File: ros2_ws/src/bot_description/urdf/robot.urdf.xacro (robot description, xacro)
@@ -19,8 +19,8 @@
     <!-- Call macros -->
     <xacro:body/>
-    <xacro:limb prefix="fl" x="${leg_x}"  y="${leg_y}"  z="${leg_z}" r="${leg_roll}" p="${leg_pitch}" yw="${leg_yaw}"  inverted_shoulder="false"/>
-    <xacro:limb prefix="fr" x="${leg_x}"  y="${-leg_y}" z="${leg_z}" r="${leg_roll}" p="${leg_pitch}" yw="${-leg_yaw}" inverted_shoulder="true" />
-    <xacro:limb prefix="bl" x="${-leg_x}" y="${leg_y}"  z="${leg_z}" r="${leg_roll}" p="${leg_pitch}" yw="${leg_yaw}"  inverted_shoulder="true" />
-    <xacro:limb prefix="br" x="${-leg_x}" y="${-leg_y}" z="${leg_z}" r="${leg_roll}" p="${leg_pitch}" yw="${-leg_yaw}" inverted_shoulder="false"/>
+    <xacro:limb prefix="fl" x="${leg_x}"  y="${leg_y}"  z="${leg_z}" r="${leg_roll}" p="${leg_pitch}" yw="${leg_yaw}"  inverted_shoulder="false" hfe_axis_mult="1" kfe_axis_mult="1"/>
+    <xacro:limb prefix="fr" x="${leg_x}"  y="${-leg_y}" z="${leg_z}" r="${leg_roll}" p="${leg_pitch}" yw="${-leg_yaw}" inverted_shoulder="true"  hfe_axis_mult="-1" kfe_axis_mult="-1"/>
+    <xacro:limb prefix="bl" x="${-leg_x}" y="${leg_y}"  z="${leg_z}" r="${leg_roll}" p="${leg_pitch}" yw="${leg_yaw}"  inverted_shoulder="true"  hfe_axis_mult="1" kfe_axis_mult="-1"/>
+    <xacro:limb prefix="br" x="${-leg_x}" y="${-leg_y}" z="${leg_z}" r="${leg_roll}" p="${leg_pitch}" yw="${-leg_yaw}" inverted_shoulder="false" hfe_axis_mult="-1" kfe_axis_mult="1"/>
      macros specific to sim/hardware modes
     <xacro:if value="$(arg sim)">
